File: current_sensor/current_sensor.kicad_sch (KiCad schematic)
At the start: 26 parts, among them Q1 S8050, Q2 S8550, U1 TL431LP, U2 TL062, U3 LM393, U4 TL062

Commit message: Finished PCB Design
Parts:
- C1, C2, C3: footprint Capacitor_THT:C_Disc_D5.0mm_W2.5mm_P2.50mm -> Capacitor_THT:C_Disc_D5.0mm_W2.5mm_P5.00mm
Connections:
- net at RV1.3: now also R1.2, U1.1 (REF)

Commit message: Final Version Ready
Parts:
- removed ADC_Current_Reading1: Conn_01x01_Socket, Connector_PinHeader_2.54mm:PinHeader_1x01_P2.54mm_Vertical, symbol Connector:Conn_01x01_Socket
- added J1: Conn_01x02_Socket, Connector_PinSocket_2.54mm:PinSocket_1x02_P2.54mm_Vertical, symbol Connector:Conn_01x02_Socket
Connections:
- net GND: now also J1.2 (Pin_2)
- net V_current_divided_clamped: now also J1.1 (Pin_1)
Changed lines of the file:
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@@
+    (stroke (width 0) (type default))
+  )
+  (wire (pts (xy 198.12 48.26) (xy 195.58 48.26))
     (stroke (width 0) (type default))
   )
@@
   )
   (wire (pts (xy 106.68 95.25) (xy 106.68 101.6))
+    (stroke (width 0) (type default))
+  )
+  (wire (pts (xy 195.58 48.26) (xy 195.58 57.15))
     (stroke (width 0) (type default))
   )
@@
     )
   )
+  (symbol (lib_id "Connector:Conn_01x02_Socket") (at 203.2 45.72 0) (unit 1)
+    (in_bom yes) (on_board yes) (dnp no) (fields_autoplaced)
+    (property "Reference" "J1" (at 204.47 45.72 0)
+      (effects (font (size 1.27 1.27)) (justify left))
+    )
+    (property "Value" "Conn_01x02_Socket" (at 204.47 48.26 0)
+      (effects (font (size 1.27 1.27)) (justify left))
+    )
+    (property "Footprint" "Connector_PinSocket_2.54mm:PinSocket_1x02_P2.54mm_Vertical" (at 203.2 45.72 0)
+      (effects (font (size 1.27 1.27)) hide)
+    )
+    (property "Datasheet" "~" (at 203.2 45.72 0)
+      (effects (font (size 1.27 1.27)) hide)
+    )
+    (pin "1")
+    (pin "2")
+    (instances
+      (project "current_sensor"
+        (path "/3057602e-8e13-4051-a806-ac2e4021c12f"
+          (reference "J1") (unit 1)
+        )
+      )
+    )
+  )
   (symbol (lib_id "power:+12V") (at 113.03 35.56 0) (unit 1)
     (in_bom yes) (on_board yes) (dnp no) (fields_autoplaced)
@@
     )
   )
+  (symbol (lib_id "power:GND") (at 195.58 57.15 0) (unit 1)
+    (in_bom yes) (on_board yes) (dnp no) (fields_autoplaced)
+    (property "Reference" "#PWR020" (at 195.58 63.5 0)
+      (effects (font (size 1.27 1.27)) hide)
+    )
+    (property "Value" "GND" (at 195.58 61.5934 0)
+      (effects (font (size 1.27 1.27)))
+    )
+    (property "Footprint" "" (at 195.58 57.15 0)
+      (effects (font (size 1.27 1.27)) hide)
+    )
+    (property "Datasheet" "" (at 195.58 57.15 0)
+      (effects (font (size 1.27 1.27)) hide)
+    )
+    (pin "1")
+    (instances
+      (project "current_sensor"
+        (path "/3057602e-8e13-4051-a806-ac2e4021c12f"
+          (reference "#PWR020") (unit 1)
+        )
+      )
+      (project "current_sensor"
+        (path "/74ccd974-f582-4f7c-bca6-79b406a1e7da"
+          (reference "#PWR019") (unit 1)
+        )
+      )
+      (project "Control_board"
+        (path "/e63e39d7-6ac0-4ffd-8aa3-1841a4541b55"
+          (reference "#PWR02") (unit 1)
+        )
+      )
+    )
+  )
   (symbol (lib_id "power:VS") (at 102.87 41.91 0) (unit 1)
     (in_bom yes) (on_board yes) (dnp no) (fields_autoplaced)
@@
         )
       )
-    )
-  )
-  (symbol (lib_id "Connector:Conn_01x01_Socket") (at 203.2 45.72 0) (unit 1)
-    (in_bom yes) (on_board yes) (dnp no) (fields_autoplaced)
-    (property "Reference" "ADC_Current_Reading1" (at 204.47 44.45 0)
-      (effects (font (size 1.27 1.27)) (justify left))
-    )
-    (property "Value" "Conn_01x01_Socket" (at 204.47 46.99 0)
-      (effects (font (size 1.27 1.27)) (justify left))
-    )
-    (property "Footprint" "Connector_PinHeader_2.54mm:PinHeader_1x01_P2.54mm_Vertical" (at 203.2 45.72 0)
-      (effects (font (size 1.27 1.27)) hide)
-    )
-    (property "Datasheet" "~" (at 203.2 45.72 0)
-      (effects (font (size 1.27 1.27)) hide)
-    )
-    (pin "1")
-    (instances
-      (project "current_sensor"
-        (path "/3057602e-8e13-4051-a806-ac2e4021c12f"
-          (reference "ADC_Current_Reading1") (unit 1)
-        )
-      )
-      (project "current_sensor"
-        (path "/74ccd974-f582-4f7c-bca6-79b406a1e7da"
-          (reference "ADC_Current_Reading1") (unit 1)
-        )
-      )
